File: Caliper_Clock_V3/Caliper_Clock_V3.kicad_sch (KiCad schematic)
At the start: 22 parts, among them J1 LCD PADS, J2 SBW, SW1 MODE, SW2 HOUR, SW3 MIN, U1 TPS61099DRVR, U2 MSP430FR4133IPM, Y1 32.768kHz

Commit message: hw: fix boost inductor rail; re-route and regen fab outputs
Fix the inductor (L1) wiring on the TPS61099 boost: it was tied to
+3V0 (VOUT) instead of +BATT (VIN), so there was no inductor path from
the cell into SW and the +3V0 rail stayed dead. Schematic now ties L1 to
+BATT. This was the root cause of the dead / 0.1 V rail (bench-confirmed
by jumpering L1 to +BATT, which brought +3V0 up to 3.0 V).

Re-route the PCB for the corrected net and regenerate Gerbers2/ + BOM/CPL
for the next fab spin.
Connections:
- net +3V0: no longer L1.1
- net +BATT: now also L1.1
Changed lines of the file:
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@@
 	)
 	(symbol
-		(lib_id "power:+3V0")
+		(lib_id "power:+BATT")
 		(at 148.59 38.1 270)
 		(unit 1)
@@
 		(on_board yes)
 		(dnp no)
-		(property "Reference" "#PWR0113"
+		(property "Reference" "#PWR04"
 			(at 143.59 38.1 0)
 			(effects
@@
 			)
 		)
-		(property "Value" "+3V0"
-			(at 157.48 37.846 90)
+		(property "Value" "+BATT"
+			(at 155.194 38.1 90)
 			(effects
 				(font
 					(size 1.27 1.27)
 				)
-				(justify right)
 			)
 		)
@@
 			(project "Caliper_Clock_V3"
 				(path "/802dda36-93fb-4ec2-b0ed-522fd3af0e85"
-					(reference "#PWR0113")
+					(reference "#PWR04")
 					(unit 1)
 				)
